File: gpib4ice.kicad_sch (KiCad schematic)
At the start: 42 parts, among them J3 Conn_02x12_Top_Bottom, U6 SN75160BN, U7 SN75161BN

Commit message: ice4pi-gpib-2.5
Parts:
- renumbered C33 to C?, C34 to C?, C7 to C?, D7 to D?, D8 to D?, J3 to J?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
