File: ice4pi.kicad_pcb (KiCad board)
At the start: 4 copper layers, 85 x 56 mm, 100 parts, among them J1 Pmod 2x6, J2 raspberry_pi_2_3_4_ordered, J3 Conn_02x12_Top_Bottom, U1 ICE40HX1K-TQ144, U2 W25Q32JVSSIQ, U3 MIC5504-1.2YM5, U4 DSC1001DI1-012.0000, U6 SN75160BN, U7 SN75161BN

Commit message: ice4pi-gpib-2.5
Parts:
- added ?: , ice4pi:mount_hole, F.Cu at (53.5, 101.5)
- added ?: , ice4pi:mount_hole, F.Cu at (111.5, 101.5)
Routing:
- net /gpib4ice/SRQ: track 14.9 -> 34.2 mm
Other:
- board text added: "ice4pi-gpib ver. 2.5"
- board text removed: "ice4pi-gpib ver. 2.4"
