File: ice4pi.kicad_sch (KiCad schematic)
At the start: 52 parts, among them J1 Pmod 2x6, J2 raspberry_pi_2_3_4_ordered, U1 ICE40HX1K-TQ144, U2 W25Q32JVSSIQ, U3 MIC5504-1.2YM5, U4 DSC1001DI1-012.0000

Commit message: ice4pi-gpib-2.5
Other:
- title: ice4pi-2.4 -> ice4pi-2.5
